Commit message: Fixed the modeling error

File: t_frog_description/urdf/t_frog.xacro (robot description, xacro)
@@ -85,23 +85,23 @@
   <link name="left_wheel">
     <collision name="collision">
-      <origin xyz="0 0.03 0" rpy="0 1.5707 1.5707"/>
-      <geometry>
-         <cylinder  length="0.05" radius="0.1"/>
+      <origin xyz="0 0.0 0" rpy="0 1.5707 1.5707"/>
+      <geometry>
+         <cylinder  length="0.03" radius="0.0725"/>
       </geometry>
     </collision>
     <visual name="visual">
-      <origin xyz="0 0.03 0" rpy="0 1.5707 1.5707"/>
-      <geometry>
-        <cylinder  length="0.05" radius="0.1"/>
+      <origin xyz="0 0.0 0" rpy="0 1.5707 1.5707"/>
+      <geometry>
+        <cylinder  length="0.03" radius="0.0725"/>
       </geometry>
     </visual>
     <inertial>
       <mass value="0.1" />
-      <origin xyz="0 0.03 0"/>
+      <origin xyz="0 0.0 0"/>
       <inertia ixx="0.1" ixy="0" ixz="0" iyy="0.1" iyz="0" izz="0.1" />
     </inertial>
   </link>
   <joint type="revolute" name="left_wheel_hinge">
-    <origin xyz="0 0.13 0.12" rpy="0 0 0"/>
+    <origin xyz="0 0.15 0.12" rpy="0 0 0"/>
     <child link="left_wheel">left_wheel</child>
     <parent link="base_link">base_link</parent>
@@ -111,23 +111,23 @@
   <link name="right_wheel">
     <collision name="collision">
-      <origin xyz="0 -0.03 0" rpy="0 1.5707 1.5707"/>
-      <geometry>
-         <cylinder  length="0.05" radius="0.1"/>
+      <origin xyz="0 0.0 0" rpy="0 1.5707 1.5707"/>
+      <geometry>
+         <cylinder  length="0.03" radius="0.0725"/>
       </geometry>
     </collision>
     <visual name="visual">
-      <origin xyz="0 -0.03 0" rpy="0 1.5707 1.5707"/>
-      <geometry>
-        <cylinder  length="0.05" radius="0.1"/>
+      <origin xyz="0 0.0 0" rpy="0 1.5707 1.5707"/>
+      <geometry>
+        <cylinder  length="0.03" radius="0.0725"/>
       </geometry>
     </visual>
     <inertial>
       <mass value="0.1" />
-      <origin xyz="0 -0.03 0"/>
+      <origin xyz="0 0.0 0"/>
       <inertia ixx="0.1" ixy="0" ixz="0" iyy="0.1" iyz="0" izz="0.1" />
     </inertial>
   </link>
   <joint type="revolute" name="right_wheel_hinge">
-    <origin xyz="0 -0.13 0.12" rpy="0 0 0"/>
+    <origin xyz="0 -0.15 0.12" rpy="0 0 0"/>
     <child link="right_wheel">right_wheel</child>
     <parent link="base_link">base_link</parent>

Commit message: Fixed a problem that the robot shakes up and down when moving

File: t_frog_description/urdf/t_frog.xacro (robot description, xacro)
@@ -21,5 +21,5 @@
       <origin xyz="0 0 0.1" rpy="0 0 0"/>
       <geometry>
-	<box size=".3 .2 .1"/>
+	<box size=".55 .4 .15"/>
       </geometry>
     </collision>
@@ -27,58 +27,24 @@
       <origin xyz="0 0 0.1" rpy="0 0 0"/>
       <geometry>
-	<box size=".3 .2 .1"/>
+	<box size=".55 .4 .15"/>
       </geometry>
       <material name="orange"/>
     </visual>
-    <collision>
-      <origin xyz="0.15 0 0.05" rpy="0 0 0"/>
+    <collision name="collision">
+      <origin xyz="-0.175 0.0 0.05" rpy="0 1.5707 1.5707"/>
       <geometry>
-	<sphere radius="0.028"/>
+         <cylinder  length="0.03" radius="0.05"/>
       </geometry>
-      <surface>
-        <friction>
-          <ode>
-	    <mu>0</mu>
-	    <mu2>0</mu2>
-	    <slip1>1.0</slip1>
-	    <slip2>1.0</slip2>
-	  </ode>
-        </friction>
-      </surface>
     </collision>
-    <visual>
-      <origin xyz="0.15 0 0.05" rpy="0 0 0"/>
+    <visual name="visual">
+      <origin xyz="-0.175 0.0 0.05" rpy="0 1.5707 1.5707"/>
       <geometry>
-	<sphere radius="0.028"/>
+        <cylinder  length="0.03" radius="0.05"/>
       </geometry>
-      <material name="orange"/>
-    </visual>
-    <collision>
-      <origin xyz="-0.15 0 0.05" rpy="0 0 0"/>
-      <geometry>
-	<sphere radius="0.028"/>
-      </geometry>
-      <surface>
-        <friction>
-          <ode>
-	    <mu>0</mu>
-	    <mu2>0</mu2>
-	    <slip1>1.0</slip1>
-	    <slip2>1.0</slip2>
-	  </ode>
-        </friction>
-      </surface>
-    </collision>
-    <visual>
-      <origin xyz="-0.15 0 0.05" rpy="0 0 0"/>
-      <geometry>
-	<sphere radius="0.028"/>
-      </geometry>
-      <material name="orange"/>
     </visual>
     <inertial>
-       <mass value="5" />
-       <origin xyz="0 0 0.1" rpy="0 0 0"/>
-       <inertia ixx="5" ixy="0" ixz="0" iyy="5" iyz="0" izz="5" />
+       <mass value="0.1" />
+       <origin xyz="0 0 0" rpy="0 0 0"/>
+       <inertia ixx="0.1" ixy="0" ixz="0" iyy="0.1" iyz="0" izz="0.1" />
     </inertial>
   </link>
@@ -97,11 +63,11 @@
     </visual>
     <inertial>
-      <mass value="0.1" />
+      <mass value="0.01" />
       <origin xyz="0 0.0 0"/>
-      <inertia ixx="0.1" ixy="0" ixz="0" iyy="0.1" iyz="0" izz="0.1" />
+      <inertia ixx="0.001" ixy="0" ixz="0" iyy="0.001" iyz="0" izz="0.001" />
     </inertial>
   </link>
   <joint type="revolute" name="left_wheel_hinge">
-    <origin xyz="0 0.15 0.12" rpy="0 0 0"/>
+    <origin xyz="0.17 0.15 0.075" rpy="0 0 0"/>
     <child link="left_wheel">left_wheel</child>
     <parent link="base_link">base_link</parent>
@@ -123,11 +89,11 @@
     </visual>
     <inertial>
-      <mass value="0.1" />
+      <mass value="0.001" />
       <origin xyz="0 0.0 0"/>
-      <inertia ixx="0.1" ixy="0" ixz="0" iyy="0.1" iyz="0" izz="0.1" />
+      <inertia ixx="0.0001" ixy="0" ixz="0" iyy="0.0001" iyz="0" izz="0.0001" />
     </inertial>
   </link>
   <joint type="revolute" name="right_wheel_hinge">
-    <origin xyz="0 -0.15 0.12" rpy="0 0 0"/>
+    <origin xyz="0.17 -0.15 0.075" rpy="0 0 0"/>
     <child link="right_wheel">right_wheel</child>
     <parent link="base_link">base_link</parent>
@@ -137,5 +103,5 @@
   <joint name="hokuyo_joint" type="fixed">
     <axis xyz="0 1 0"/>
-    <origin xyz="0.15 0 0.175" rpy="0 0 0"/>
+    <origin xyz="0.275 0 0.2" rpy="0 0 0"/>
     <parent link="base_link"/>
     <child link="hokuyo_link"/>
@@ -155,12 +121,12 @@
     </visual>
     <inertial>
-      <mass value="1"/>
+      <mass value="0.0001"/>
       <origin xyz="0 0 0" rpy="0 0 0"/>
-      <inertia ixx="1" ixy="0" ixz="0" iyy="1" iyz="0" izz="1"/>
+      <inertia ixx="0.0001" ixy="0" ixz="0" iyy="0.0001" iyz="0" izz="0.0001"/>
     </inertial>
   </link>
   <joint name="camera_joint" type="fixed">
     <axis xyz="0 1 0" />
-    <origin xyz="-0.15 0 0.175" rpy="0 0 0"/>
+    <origin xyz="-0.275 0 0.2" rpy="0 0 0"/>
     <parent link="base_link"/>
     <child link="camera_link"/>
@@ -181,7 +147,7 @@
     </visual>
     <inertial>
-      <mass value="1"/>
+      <mass value="0.0001"/>
       <origin xyz="0 0 0" rpy="0 0 0"/>
-      <inertia ixx="1" ixy="0" ixz="0" iyy="1" iyz="0" izz="1"/>
+      <inertia ixx="0.0001" ixy="0" ixz="0" iyy="0.0001" iyz="0" izz="0.0001"/>
     </inertial>
   </link>

Commit message: Equalize the mass of the left and right

File: t_frog_description/urdf/t_frog.xacro (robot description, xacro)
@@ -89,7 +89,7 @@
     </visual>
     <inertial>
-      <mass value="0.001" />
+      <mass value="0.01" />
       <origin xyz="0 0.0 0"/>
-      <inertia ixx="0.0001" ixy="0" ixz="0" iyy="0.0001" iyz="0" izz="0.0001" />
+      <inertia ixx="0.001" ixy="0" ixz="0" iyy="0.001" iyz="0" izz="0.001" />
     </inertial>
   </link>

Commit message: 旋回性能が極端に悪い問題に対して暫定対処

File: t_frog_description/urdf/t_frog.xacro (robot description, xacro)
@@ -34,5 +34,5 @@
       <origin xyz="-0.175 0.0 0.05" rpy="0 1.5707 1.5707"/>
       <geometry>
-         <cylinder  length="0.03" radius="0.05"/>
+        <cylinder  length="0.03" radius="0.05"/>
       </geometry>
     </collision>
@@ -44,7 +44,7 @@
     </visual>
     <inertial>
-       <mass value="0.1" />
+       <mass value="20" />
        <origin xyz="0 0 0" rpy="0 0 0"/>
-       <inertia ixx="0.1" ixy="0" ixz="0" iyy="0.1" iyz="0" izz="0.1" />
+       <inertia ixx="1" ixy="0" ixz="0" iyy="1" iyz="0" izz="1" />
     </inertial>
   </link>
@@ -63,15 +63,15 @@
     </visual>
     <inertial>
-      <mass value="0.01" />
+      <mass value="1" />
       <origin xyz="0 0.0 0"/>
-      <inertia ixx="0.001" ixy="0" ixz="0" iyy="0.001" iyz="0" izz="0.001" />
+      <inertia ixx="0.1" ixy="0" ixz="0" iyy="0.1" iyz="0" izz="0.1" />
     </inertial>
   </link>
   <joint type="revolute" name="left_wheel_hinge">
-    <origin xyz="0.17 0.15 0.075" rpy="0 0 0"/>
+    <origin xyz="0 0.15 0.075" rpy="0 0 0"/>
     <child link="left_wheel">left_wheel</child>
     <parent link="base_link">base_link</parent>
     <axis xyz="0 1 0"/>
-    <limit effort="30" velocity="1.0"  lower="-100" upper="100" />
+    <limit effort="100" velocity="100.0"  lower="-1000" upper="1000" />
   </joint>
   <link name="right_wheel">
@@ -89,15 +89,15 @@
     </visual>
     <inertial>
-      <mass value="0.01" />
+      <mass value="1" />
       <origin xyz="0 0.0 0"/>
-      <inertia ixx="0.001" ixy="0" ixz="0" iyy="0.001" iyz="0" izz="0.001" />
+      <inertia ixx="0.1" ixy="0" ixz="0" iyy="0.1" iyz="0" izz="0.1" />
     </inertial>
   </link>
   <joint type="revolute" name="right_wheel_hinge">
-    <origin xyz="0.17 -0.15 0.075" rpy="0 0 0"/>
+    <origin xyz="0 -0.15 0.075" rpy="0 0 0"/>
     <child link="right_wheel">right_wheel</child>
     <parent link="base_link">base_link</parent>
     <axis xyz="0 1 0"/>
-    <limit effort="30" velocity="1.0"  lower="-100" upper="100" />
+    <limit effort="100" velocity="100.0"  lower="-1000" upper="1000" />
   </joint>
   <joint name="hokuyo_joint" type="fixed">

Commit message: Added the virtual links

File: t_frog_description/urdf/t_frog.xacro (robot description, xacro)
@@ -34,5 +34,5 @@
       <origin xyz="-0.175 0.0 0.05" rpy="0 1.5707 1.5707"/>
       <geometry>
-        <cylinder  length="0.03" radius="0.05"/>
+        <cylinder  length="0.03" radius="0.04625"/>
       </geometry>
     </collision>
@@ -40,7 +40,13 @@
       <origin xyz="-0.175 0.0 0.05" rpy="0 1.5707 1.5707"/>
       <geometry>
-        <cylinder  length="0.03" radius="0.05"/>
-      </geometry>
-    </visual>
+        <cylinder  length="0.03" radius="0.04625"/>
+      </geometry>
+    </visual>
+    <collision name="collision">
+      <origin xyz="0.175 0.0 0.05" rpy="0 1.5707 1.5707"/>
+      <geometry>
+        <cylinder  length="0.03" radius="0.04625"/>
+      </geometry>
+    </collision>
     <inertial>
        <mass value="20" />
@@ -49,4 +55,18 @@
     </inertial>
   </link>
+  <link name="visual_left_wheel">
+    <visual name="visual">
+      <origin xyz="0 0.0 0" rpy="0 1.5707 1.5707"/>
+      <geometry>
+        <cylinder  length="0.03" radius="0.0725"/>
+      </geometry>
+    </visual>
+  </link>
+  <joint type="fixed" name="visual_left_wheel_hinge">
+    <origin xyz="0.15 0.15 0.075" rpy="0 0 0"/>
+    <child link="visual_left_wheel">visual_left_wheel</child>
+    <parent link="base_link">base_link</parent>
+    <axis xyz="0 1 0"/>
+  </joint>
   <link name="left_wheel">
     <collision name="collision">
@@ -56,10 +76,10 @@
       </geometry>
     </collision>
-    <visual name="visual">
-      <origin xyz="0 0.0 0" rpy="0 1.5707 1.5707"/>
-      <geometry>
-        <cylinder  length="0.03" radius="0.0725"/>
-      </geometry>
-    </visual>
+    <!--visual name="visual">
+      <origin xyz="0 0.0 0" rpy="0 1.5707 1.5707"/>
+      <geometry>
+        <cylinder  length="0.03" radius="0.0725"/>
+      </geometry>
+    </visual-->
     <inertial>
       <mass value="1" />
@@ -75,4 +95,18 @@
     <limit effort="100" velocity="100.0"  lower="-1000" upper="1000" />
   </joint>
+  <link name="visual_right_wheel">
+    <visual name="visual">
+      <origin xyz="0 0.0 0" rpy="0 1.5707 1.5707"/>
+      <geometry>
+        <cylinder  length="0.03" radius="0.0725"/>
+      </geometry>
+    </visual>
+  </link>
+  <joint type="fixed" name="visual_right_wheel_hinge">
+    <origin xyz="0.15 -0.15 0.075" rpy="0 0 0"/>
+    <child link="visual_right_wheel">visual_right_wheel</child>
+    <parent link="base_link">base_link</parent>
+    <axis xyz="0 1 0"/>
+  </joint>
   <link name="right_wheel">
     <collision name="collision">
@@ -82,10 +116,10 @@
       </geometry>
     </collision>
-    <visual name="visual">
-      <origin xyz="0 0.0 0" rpy="0 1.5707 1.5707"/>
-      <geometry>
-        <cylinder  length="0.03" radius="0.0725"/>
-      </geometry>
-    </visual>
+    <!--visual name="visual">
+      <origin xyz="0 0.0 0" rpy="0 1.5707 1.5707"/>
+      <geometry>
+        <cylinder  length="0.03" radius="0.0725"/>
+      </geometry>
+    </visual-->
     <inertial>
       <mass value="1" />

Commit message: Fixed upper limits of the amount of movement

File: t_frog_description/urdf/t_frog.xacro (robot description, xacro)
@@ -93,5 +93,5 @@
     <parent link="base_link">base_link</parent>
     <axis xyz="0 1 0"/>
-    <limit effort="100" velocity="100.0"  lower="-1000" upper="1000" />
+    <limit effort="100" velocity="100.0"  lower="-5000" upper="5000" />
   </joint>
   <link name="visual_right_wheel">
@@ -133,5 +133,5 @@
     <parent link="base_link">base_link</parent>
     <axis xyz="0 1 0"/>
-    <limit effort="100" velocity="100.0"  lower="-1000" upper="1000" />
+    <limit effort="100" velocity="100.0"  lower="-5000" upper="5000" />
   </joint>
   <joint name="hokuyo_joint" type="fixed">
