Commit message: Change the project name from t_frog_driver to icart_mini_driver

File: icart_mini_description/urdf/icart_mini.xacro (robot description, xacro)
@@ -1,5 +1,5 @@
 <?xml version="1.0"?>
 <!-- Revolute-Revolute Manipulator -->
-<robot name="t_frog" xmlns:xacro="http://www.ros.org/wiki/xacro">
+<robot name="icart_mini" xmlns:xacro="http://www.ros.org/wiki/xacro">
   <!-- Constants for robot dimensions -->
   <xacro:property name="PI" value="3.1415926535897931"/>
@@ -7,7 +7,7 @@
   <xacro:property name="hokuyo_link" value="0.1" /> <!-- Size of square 'hokuyo' box -->
   <!-- Import all Gazebo-customization elements, including Gazebo colors -->
-  <xacro:include filename="$(find t_frog_description)/urdf/t_frog.gazebo" />
+  <xacro:include filename="$(find icart_mini_description)/urdf/icart_mini.gazebo" />
   <!-- Import Rviz colors -->
-  <xacro:include filename="$(find t_frog_description)/urdf/materials.xacro" />
+  <xacro:include filename="$(find icart_mini_description)/urdf/materials.xacro" />
   <!-- Used for fixing robot to Gazebo 'base_link' -->
   <!--link name="world"/>
@@ -151,5 +151,5 @@
       <origin xyz="0 0 0" rpy="0 0 0"/>
       <geometry>
-        <mesh filename="package://t_frog_description/meshes/hokuyo.dae"/>
+        <mesh filename="package://icart_mini_description/meshes/hokuyo.dae"/>
       </geometry>
     </visual>

Commit message: Correspond to the new exterior of the i-Cart mini

File: icart_mini_description/urdf/icart_mini.xacro (robot description, xacro)
@@ -21,5 +21,5 @@
       <origin xyz="0 0 0.1" rpy="0 0 0"/>
       <geometry>
-	<box size=".55 .4 .15"/>
+	<box size=".485 .43 .15"/>
       </geometry>
     </collision>
@@ -27,5 +27,5 @@
       <origin xyz="0 0 0.1" rpy="0 0 0"/>
       <geometry>
-	<box size=".55 .4 .15"/>
+	<box size=".485 .43 .15"/>
       </geometry>
       <material name="orange"/>
@@ -137,5 +137,5 @@
   <joint name="hokuyo_joint" type="fixed">
     <axis xyz="0 1 0"/>
-    <origin xyz="0.275 0 0.2" rpy="0 0 0"/>
+    <origin xyz="0.243 0 0.2" rpy="0 0 0"/>
     <parent link="base_link"/>
     <child link="hokuyo_link"/>
@@ -162,5 +162,5 @@
   <joint name="camera_joint" type="fixed">
     <axis xyz="0 1 0" />
-    <origin xyz="-0.275 0 0.2" rpy="0 0 0"/>
+    <origin xyz="0 0 0.2" rpy="0 0 0"/>
     <parent link="base_link"/>
     <child link="camera_link"/>
